File: mcu.kicad_sch (KiCad schematic)
At the start: 14 parts, among them U1 STM32G071C8Tx, Y1 NX3225GD

Commit message: Fix xtal circuit
Parts:
- removed R23, R24: 100R, symbol Device:R
- C29, C30: value 10pF -> 14pF
- Y1: value NX3225GD -> NX3215SA-32.768K-STD-MUA-9; JLCPCB Part No C889706 -> C519280
Connections:
- net at C30.2, Y1.1: now also U1.9 (PF1)
- net at C29.2, Y1.2: now also U1.8 (PF0)
Other:
- note removed: "TODO: Check R23, R24 (maybe not needed), calculate C29 and C30"
- note removed: "TODO: verify i2c pullup resistance value"
Changed lines of the file:
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@@
 	(wire
 		(pts
-			(xy 68.58 78.74) (xy 73.66 78.74)
+			(xy 68.58 78.74) (xy 83.82 78.74)
 		)
 		(stroke
@@
 	(wire
 		(pts
-			(xy 83.82 69.85) (xy 81.28 69.85)
-		)
-		(stroke
-			(width 0)
-			(type default)
-		)
-	)
-	(wire
-		(pts
 			(xy 58.42 167.64) (xy 69.85 167.64)
 		)
@@
 	(wire
 		(pts
-			(xy 83.82 78.74) (xy 81.28 78.74)
-		)
-		(stroke
-			(width 0)
-			(type default)
-		)
-	)
-	(wire
-		(pts
 			(xy 171.45 134.62) (xy 171.45 133.35)
 		)
@@
 	(wire
 		(pts
-			(xy 68.58 69.85) (xy 73.66 69.85)
+			(xy 68.58 69.85) (xy 83.82 69.85)
 		)
 		(stroke
@@
 		)
 	)
-	(text "TODO: verify i2c pullup resistance value"
-		(exclude_from_sim no)
-		(at 190.5 133.35 0)
-		(effects
-			(font
-				(size 1.27 1.27)
-			)
-			(justify left bottom)
-		)
-	)
 	(text "- ST32G0 UDPD: https://www.st.com/resource/en/product_training/STM32G0-Peripheral-USB-Type-C-Power-Delivery-UCPD.pdf\n"
 		(exclude_from_sim no)
@@
 			(justify left bottom)
 			(href "https://www.st.com/resource/en/product_training/STM32G0-Peripheral-USB-Type-C-Power-Delivery-UCPD.pdf")
-		)
-	)
-	(text "TODO: Check R23, R24 (maybe not needed), calculate C29 and C30\n"
-		(exclude_from_sim no)
-		(at 60.706 59.944 0)
-		(effects
-			(font
-				(size 1.27 1.27)
-			)
 		)
 	)
@@
 	)
 	(symbol
-		(lib_id "Device:R")
-		(at 77.47 78.74 90)
-		(mirror x)
-		(unit 1)
-		(exclude_from_sim no)
-		(in_bom yes)
-		(on_board yes)
-		(dnp no)
-		(property "Reference" "R24"
-			(at 77.47 85.09 90)
-			(effects
-				(font
-					(size 1.27 1.27)
-				)
-			)
-		)
-		(property "Value" "100R"
-			(at 77.47 82.55 90)
-			(effects
-				(font
-					(size 1.27 1.27)
-				)
-			)
-		)
-		(property "Footprint" ""
-			(at 77.47 76.962 90)
-			(effects
-				(font
-					(size 1.27 1.27)
-				)
-				(hide yes)
-			)
-		)
-		(property "Datasheet" "~"
-			(at 77.47 78.74 0)
-			(effects
-				(font
-					(size 1.27 1.27)
-				)
-				(hide yes)
-			)
-		)
-		(property "Description" ""
-			(at 77.47 78.74 0)
-			(effects
-				(font
-					(size 1.27 1.27)
-				)
-				(hide yes)
-			)
-		)
-		(property "LCSC Part No" ""
-			(at 77.47 78.74 0)
-			(effects
-				(font
-					(size 1.27 1.27)
-				)
-				(hide yes)
-			)
-		)
-		(property "JLCPCB Part No" ""
-			(at 77.47 78.74 0)
-			(effects
-				(font
-					(size 1.27 1.27)
-				)
-				(hide yes)
-			)
-		)
-		(property "V_{max}" ""
-			(at 77.47 78.74 0)
-			(effects
-				(font
-					(size 1.27 1.27)
-				)
-			)
-		)
-		(pin "1"
-		)
-		(pin "2"
-		)
-		(instances
-			(project "usb-zekers"
-				(path "/1eef11ed-4055-4fe6-b7fc-0d497914d6cc/c7a7dbb8-992c-4c2f-932e-320edf489341"
-					(reference "R24")
-					(unit 1)
-				)
-			)
-		)
-	)
-	(symbol
 		(lib_id "Device:C")
 		(at 45.72 172.72 0)
@@
 				(path "/1eef11ed-4055-4fe6-b7fc-0d497914d6cc/c7a7dbb8-992c-4c2f-932e-320edf489341"
 					(reference "C22")
-					(unit 1)
-				)
-			)
-		)
-	)
-	(symbol
-		(lib_id "Device:R")
-		(at 77.47 69.85 90)
-		(unit 1)
-		(exclude_from_sim no)
-		(in_bom yes)
-		(on_board yes)
-		(dnp no)
-		(fields_autoplaced yes)
-		(property "Reference" "R23"
-			(at 77.47 63.5 90)
-			(effects
-				(font
-					(size 1.27 1.27)
-				)
-			)
-		)
-		(property "Value" "100R"
-			(at 77.47 66.04 90)
-			(effects
-				(font
-					(size 1.27 1.27)
-				)
-			)
-		)
-		(property "Footprint" ""
-			(at 77.47 71.628 90)
-			(effects
-				(font
-					(size 1.27 1.27)
-				)
-				(hide yes)
-			)
-		)
-		(property "Datasheet" "~"
-			(at 77.47 69.85 0)
-			(effects
-				(font
-					(size 1.27 1.27)
-				)
-				(hide yes)
-			)
-		)
-		(property "Description" ""
-			(at 77.47 69.85 0)
-			(effects
-				(font
-					(size 1.27 1.27)
-				)
-				(hide yes)
-			)
-		)
-		(property "LCSC Part No" ""
-			(at 77.47 69.85 0)
-			(effects
-				(font
-					(size 1.27 1.27)
-				)
-				(hide yes)
-			)
-		)
-		(property "JLCPCB Part No" ""
-			(at 77.47 69.85 0)
-			(effects
-				(font
-					(size 1.27 1.27)
-				)
-				(hide yes)
-			)
-		)
-		(property "V_{max}" ""
-			(at 77.47 69.85 0)
-			(effects
-				(font
-					(size 1.27 1.27)
-				)
-			)
-		)
-		(pin "2"
-		)
-		(pin "1"
-		)
-		(instances
-			(project "usb-zekers"
-				(path "/1eef11ed-4055-4fe6-b7fc-0d497914d6cc/c7a7dbb8-992c-4c2f-932e-320edf489341"
-					(reference "R23")
 					(unit 1)
 				)
@@
 			)
 		)
-		(property "Value" "10pF"
+		(property "Value" "14pF"
 			(at 59.69 64.77 90)
 			(effects
@@
 			)
 		)
-		(property "Value" "NX3225GD"
+		(property "Value" "   NX3215SA-32.768K-STD-MUA-9"
 			(at 66.04 74.93 90)
 			(effects
@@
 			)
 		)
-		(property "JLCPCB Part No" "C889706"
+		(property "JLCPCB Part No" "C519280"
 			(at 68.58 73.66 0)
 			(effects
@@
 			)
 		)
-		(property "Value" "10pF"
+		(property "Value" "14pF"
 			(at 59.69 83.82 90)
 			(effects
